File: lightrail-lpo-mvp-repaired/LightRail_LPO_MVP.kicad_pcb (KiCad board)
At the start: 2 copper layers, 15 parts, among them J1 SMA, J2 SMA, J3 SMA, J4 SMA, U1 TFLN-MZM-400G-C, U2 TLN-1550-100, U3 XPDV4120R, U4 HMC8410

Commit message: Auto-generate native KiCad 10.0 Gerber and Drill files for LPO MVP and LR-P3A Rev 6.3 after fixing stackup and pad syntax compatibility
Other:
- board outline added: 295 x 140 mm
- net class Default added: clearance 0.2, trace_width 0.25, via_dia 0.8, via_drill 0.4
