File: 15_lr_p3a_datasheet_design/kicad/LR_P3A_DualNCE.kicad_pcb (KiCad board)
At the start: 16 copper layers, 230 x 150 mm, 12 parts, among them U102 TFLN-MZM-400G-C, U202 TFLN-MZM-400G-C

Commit message: Auto-route Phase 1 differential pairs and pour plane layers
Routing:
- net PCIE_G6_B: track 0.00 -> 114.4 mm
- net PCIE_G6_A: track 0.00 -> 114.4 mm
- net SERDES_200G_B: track 0.00 -> 76.0 mm
- net SERDES_200G_A: track 0.00 -> 76.0 mm
- net TFLN_RF_B: track 0.00 -> 5.62 mm
- net TFLN_RF_A: track 0.00 -> 5.62 mm
- added copper zone on In7.Cu, net GND
- added copper zone on In12.Cu, net PWR_CORE

Commit message: Route all Phase 2 secondary nets using orthogonal BGA comb routing
Routing:
- net HBM4_SIDECH_B: track 0.00 -> 24.8 mm
- net HBM4_SIDECH_A: track 0.00 -> 24.8 mm
- net MGMT_A: track 0.00 -> 24.8 mm
- net MGMT_B: track 0.00 -> 24.8 mm
- net PD_MON_B: track 0.00 -> 2.62 mm
- net PD_MON_A: track 0.00 -> 2.62 mm
- net BIAS_TUNE_B: track 0.00 -> 2.62 mm
- net BIAS_TUNE_A: track 0.00 -> 2.62 mm
