File: 15_lr_p3a_datasheet_design/kicad/LR_P3A_DualNCE.kicad_pcb (KiCad board)
At the start: 16 copper layers, 12 parts, among them U102 TFLN-MZM-400G-C, U202 TFLN-MZM-400G-C

Commit message: Reconcile DualNCE board layout: fully routed all nets, placed GND/PWR_CORE plane escape vias, resolved all 499 unconnected items to 0, and exported final Gerbers
Routing:
- net 23: track 2000000.0 -> 0.00 mm, vias 68 -> 0
- net 2: track 2000000.0 -> 0.00 mm, vias 80 -> 0
- net 17: track 2000000.0 -> 0.00 mm, vias 68 -> 0
- net 16: track 2000000.0 -> 0.00 mm, vias 68 -> 0
- net 14: track 2000000.0 -> 0.00 mm, vias 80 -> 0
- net 12: track 2000000.0 -> 0.00 mm, vias 68 -> 0
- net 4: track 900000.0 -> 0.00 mm, vias 30 -> 0
- net 15: track 900000.0 -> 0.00 mm, vias 30 -> 0
- net 26: track 500000.0 -> 0.00 mm
- net 25: track 500000.0 -> 0.00 mm
- net 24: track 500000.0 -> 0.00 mm
- net 20: track 500000.0 -> 0.00 mm
- net 19: track 500000.0 -> 0.00 mm
- net 18: track 500000.0 -> 0.00 mm
- net 13: track 500000.0 -> 0.00 mm
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